File: kicad/DC_Amplifier.kicad_pcb (KiCad board)
At the start: 2 copper layers, 61 x 35.6 mm, 18 parts, among them J1 Conn_01x03, U1 OPAMP

Commit message: kicad 7
Other:
- net class Default removed
- board text added: "REVISION B JULY 2023"
- board text removed: "REVISION 1.1.0 FEBRUARY 2021"
